File: KiCad/Ceiling lamp/Ceiling lamp.kicad_pcb (KiCad board)
At the start: 2 copper layers, 49.5 x 49.5 mm, 16 parts, among them J1 Screw_Terminal_01x04, J2 Conn_01x06_Female, K1 1461492-2, Q1 FDN537N, SW1 SW_Push, U1 BU33SD5WG-TR, U2 ESP-12E, U3 HLK-PM01

Commit message: pcb changes v3
Other:
- board text added: "AC in"
- board text added: "AC out"
- board text added: "Ceiling lamp - ESP8266 Design by Enrique Gómez CC BY-SA 4.0 www.rinconingenieril.es Rev.: 3.0 - S/N:"
- board text added: "GND 3.3v Fla Rst RX TX"
- board text removed: "Ceiling lamp - ESP8266 Design by Enrique Gómez CC BY-SA 4.0 www.rinconingenieril.es Rev.: 2.0 - S/N:"
